File: board/board.kicad_pcb (KiCad board)
At the start: 2 copper layers, 21 x 13 mm, 1 part

Commit message: added LCSC Part numbers
Parts:
- added C1: 100pF, Capacitor_SMD:C_0402_1005Metric, F.Cu at (148.0, 92.0)
- added J1: C3020043, b142:TYPE-C 16PFS 4J-H7.05 IPX6, F.Cu at (143.0, 96.5)
- added J2: 008_USB, on_edge:on_edge_2x05_host, F.Cu at (161.0, 96.5)
- added R1: 5.1k, Resistor_SMD:R_0402_1005Metric, F.Cu at (148.0, 94.0)
- added R2: 5.1k, Resistor_SMD:R_0402_1005Metric, F.Cu at (148.0, 99.0)
- added R3: 0R, Resistor_SMD:R_0603_1608Metric, F.Cu at (154.2, 94.5)
- added R4: 0R, Resistor_SMD:R_0603_1608Metric, F.Cu at (154.2, 96.0)
- moved LOGO1 2.06 mm to (152.0, 99.5)
Routing:
- net GND: track 0.00 -> 24.3 mm, vias 0 -> 2
- net Net-(C1-Pad1): track 0.00 -> 19.3 mm
- net /usb-c/DM: track 0.00 -> 16.2 mm
- net /usb-c/VBUS: track 0.00 -> 16.1 mm, vias 0 -> 2
- net /usb-c/DP: track 0.00 -> 14.8 mm, vias 0 -> 2
- net Net-(J2-5V): track 0.00 -> 7.74 mm, vias 0 -> 1
- net Net-(J2-VBUS): track 0.00 -> 3.65 mm
- net Net-(J1-CC1): track 0.00 -> 2.21 mm
- net Net-(J1-CC2): track 0.00 -> 1.99 mm
Other:
- outline, holes or cut-outs redrawn
- board text added: "osf.008"
- board text added: "osf.b142.v1.0"
